File: hardware/Rev_B/FT2D_PD20V_12V5_3A_评审原理图.kicad_pcb (KiCad board)
At the start: 4 copper layers, 105 x 65 mm, 58 parts, among them J1 USB4085-GF-A, J2 PD_PROGRAM_TEST, J3 E-DC-6_PIGTAIL, Q1 STL6P3LLH6, U1 STUSB4500QTR, U2 LM61460AASQRJRRQ1, U3 TPS259474ARPWR

Commit message: Rev B: verify JLC SMT J1/L1, tighten buck routing and audit 3A/GND (NO-GO)
Parts:
- J1: value USB4085-GF-A -> TYPE-C-31-M-12; footprint Connector_USB:USB_C_Receptacle_GCT_USB4085 -> Connector_USB:USB_C_Receptacle_HRO_TYPE-C-31-M-12
- L1: value SRP1238A-100M_10uH -> SRG1260-100-M_10uH; footprint FT2D:Bourns_SRP1238A -> FT2D:JIERR_SRG1260_100M
- moved C12 8.00 mm to (77.0, 38.0)
- moved U2 7.00 mm to (79.0, 43.0)
- moved C19 4.03 mm to (79.0, 48.5)
- moved R19 3.00 mm to (74.0, 48.0)
- moved C13 2.00 mm to (73.0, 38.0)
- moved J1 0.85 mm to (24.1, 42.0), turned to -90 degrees
Routing:
- net /VBUS_SW: track 89.1 -> 76.4 mm, vias 3 -> 2
- net /SCL: track 34.8 -> 47.3 mm
- net /CC1: track 37.2 -> 26.1 mm
- net /V12P5: track 105.5 -> 96.9 mm
- net /VBUS_RAW: track 81.0 -> 89.6 mm, vias 2 -> 0
- net /VBUS_EN_SNK: track 21.5 -> 14.2 mm, vias 2 -> 0
- net /USB_VBUS: track 23.2 -> 16.2 mm, vias 2 -> 0
- net /BUCK_VCC: track 9.94 -> 15.1 mm
- net /PD_RESET: track 49.7 -> 45.1 mm
- net /PGTH_U3: track 19.0 -> 23.3 mm, vias 2 -> 0
- net /BUCK_RT: track 6.84 -> 11.2 mm
- net /PD_1V2: track 7.17 -> 11.3 mm, vias 2 -> 0
- net /BUCK_PGOOD: track 10.4 -> 14.2 mm
- net /FB_U2: track 25.6 -> 22.0 mm, vias 0 -> 2
- net /PD_GATE: track 17.6 -> 20.8 mm, vias 2 -> 3
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- added copper zone on F.Cu, net /SW
- added copper zone on F.Cu, net /USB_VBUS
- added copper zone on F.Cu, net /V12P5
- added copper zone on F.Cu, net /VBUS_RAW
- added copper zone on F.Cu, net /VBUS_SW
- added copper zone on F.Cu, net /VOUT

Commit message: Rev B: clear ERC/DRC/GND, validate C18 JLC hybrid footprint, export QA Gerbers and SMT sourcing review (NO-GO)
Parts:
- C18: value EEHZL1V470R_47u -> EEHZA1V470P_47u; footprint Capacitor_SMD:CP_Elec_5x5.8 -> Capacitor_SMD:CP_Elec_6.3x5.8
- moved C18 0.50 mm to (61.5, 48.0)
Routing:
- net /GND: track 0.00 -> 13.9 mm, vias 7 -> 15
- net /SCL: track 47.3 -> 35.8 mm
- net /ILM_U3: track 22.7 -> 30.7 mm
- net /PG_U3: track 13.1 -> 20.7 mm, vias 2 -> 0
- net /SDA: track 36.9 -> 42.7 mm
- net /CC1: track 26.1 -> 31.8 mm
- net /VOUT: track 48.9 -> 43.5 mm
- net /PGTH_U3: track 23.3 -> 19.0 mm, vias 0 -> 2
- net /VBUS_EN_SNK: track 14.2 -> 18.4 mm, vias 0 -> 2
- net /V12P5: track 96.9 -> 100.7 mm
- net /BUCK_VCC: track 15.1 -> 18.7 mm
- net /PD_2V7: track 50.3 -> 53.7 mm, vias 4 -> 3
- net /ITIMER_U3: track 8.42 -> 11.5 mm, vias 0 -> 2
- net /PD_GATE: track 20.8 -> 23.4 mm, vias 3 -> 2
- net /PD_DISCH: track 10.1 -> 7.75 mm, vias 2 -> 0
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
Commit message: Rev B: stitch U3 power copper and upgrade output bypass; refresh JLC review QA (NO-GO)
Parts:
- C26: value 100n_25V -> 2u2_25V
Routing:
- net /VOUT: vias 0 -> 2
- net /V12P5: vias 0 -> 2
- added copper zone on In2.Cu, net /V12P5
- added copper zone on In2.Cu, net /VOUT
Changed lines of the file:
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@@
 			)
 		)
-		(property "Value" "100n_25V"
+		(property "Value" "2u2_25V"
 			(at 0 1.43 0)
 			(layer "F.Fab")
@@
 		(net "/V12P5")
 	)
+	(via
+		(at 104 44.1)
+		(size 0.6)
+		(drill 0.3)
+		(layers "F.Cu" "B.Cu")
+		(net "/V12P5")
+	)
+	(via
+		(at 104 45)
+		(size 0.6)
+		(drill 0.3)
+		(layers "F.Cu" "B.Cu")
+		(net "/V12P5")
+	)
 	(segment
 		(start 81.6059 46.6691)
@@
 		(net "/VOUT")
 	)
+	(via
+		(at 111 45)
+		(size 0.6)
+		(drill 0.3)
+		(layers "F.Cu" "B.Cu")
+		(net "/VOUT")
+	)
+	(via
+		(at 115 44)
+		(size 0.6)
+		(drill 0.3)
+		(layers "F.Cu" "B.Cu")
+		(net "/VOUT")
+	)
 	(segment
 		(start 102.908 43.225)
@@
 			)
 		)
+	)
+	(zone
+		(net "/V12P5")
+		(layer "In2.Cu")
+		(name "REV_B_U3_IN2_V12P5")
+		(hatch edge 0.5)
+		(priority 2)
+		(connect_pads yes
+			(clearance 0.3)
+		)
+		(min_thickness 0.25)
+		(fill yes
+			(thermal_gap 0.5)
+			(thermal_bridge_width 0.5)
+			(island_removal_mode 0)
+		)
+		(polygon
+			(pts
+				(xy 102 39) (xy 108.1 39) (xy 108.1 48.2) (xy 102 48.2)
+			)
+		)
+	)
+	(zone
+		(net "/VOUT")
+		(layer "In2.Cu")
+		(name "REV_B_U3_IN2_VOUT")
+		(hatch edge 0.5)
+		(priority 2)
+		(connect_pads yes
+			(clearance 0.3)
+		)
+		(min_thickness 0.25)
+		(fill yes
+			(thermal_gap 0.5)
+			(thermal_bridge_width 0.5)
+			(island_removal_mode 0)
+		)
+		(polygon
+			(pts
+				(xy 109.2 39) (xy 116 39) (xy 116 48.2) (xy 109.2 48.2)
+			)
+		)

Commit message: Rev B: qualify JLC SMT 102k OVLO resistor and refresh fab preview artifacts (NO-GO)
Parts:
- R22: value 101k -> 102k
Changed lines of the file:
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@@
 			)
 		)
-		(property "Value" "101k"
+		(property "Value" "102k"
 			(at 0 1.43 0)
 			(layer "F.Fab")
